File: HapticsFinal/HapticsFinal.kicad_pcb (KiCad board)
At the start: 2 copper layers, 35.8 x 44.5 mm, 41 parts, among them IC4 TPS62142RGTR, IC5 TPS62153RGTR, J1 Conn_01x04_Pin, J2 Conn_01x06_Pin, J3 Conn_01x03_Pin, J4 Conn_01x04_Pin, Q1 AO3400A, Q2 AO3400A, Q3 AO3400A, U2 ESP32-C3-SuperMini

Commit message: reviewed board : Changed Silkscreen for readability and cleared ERC & DRC errors
Parts:
- moved C12 0.19 mm to (131.0, 107.0)
- turned R8 to 0 degrees
Connections:
- C10 pad 2: 3.3V -> M1out1
- C3 pad 1: 3.3V -> M1out1
- C4 pad 1: 3.3V -> M1out1
- C5 pad 1: 3.3V -> M1out1
- D4 pad 1: 3.3V -> M1out1
- D5 pad 1: 3.3V -> M1out1
- D6 pad 1: 3.3V -> M1out1
- IC4 pad 14: 3.3V -> M1out1
- IC4 pad 7: 3.3V -> M1out1
- J2 pad 2: 3.3V -> M1out1
- J2 pad 3: 3.3V -> M1out1
- J2 pad 5: 3.3V -> M1out1
- L2 pad 1: 3.3V -> M1out1
- R4 pad 1: 3.3V -> M1out1
- R5 pad 1: 3.3V -> M1out1
- R8 pad 1: Net-(Q1-G) -> M1in
- R8 pad 2: M1in -> Net-(Q1-G)
- U2 pad 3V3: (no net) -> unconnected-(U2-Pad3V3)
- U2 pad 5V: (no net) -> M1out1
- U2 pad GND: (no net) -> GND
Routing:
- net M1out1: track 0.00 -> 120.3 mm, vias 0 -> 11
- net 3.3V: track 95.3 -> 0.00 mm, vias 5 -> 0
- net GND: track 46.9 -> 51.4 mm, vias 13 -> 15
Other:
- board text added: "+3.3V Power"
- board text added: "+5V Power"
- board text removed: "+3.3V"
- board text removed: "+5V"
- board text removed: "Power/Temp"
