File: HapticsFinal/HapticsFinal.kicad_sch (KiCad schematic)
At the start: 40 parts, among them IC4 TPS62142RGTR, IC5 TPS62153RGTR, J1 Conn_01x04_Pin, J2 Conn_01x06_Pin, J3 Conn_01x03_Pin, J4 Conn_01x04_Pin, Q1 AO3400A, Q2 AO3400A, Q3 AO3400A, U2 ESP32-C3-SuperMini

Commit message: reviewed board : Changed Silkscreen for readability and cleared ERC & DRC errors
Connections:
- net +3.3V: now also U2.5V; no longer U2. (3V3)
- net GND: now also U2.GND; no longer U2. (3V3)
- net M1in: now also R8.1; no longer R8.2
- net at Q1.1 (G), R7.1: now also R8.2; no longer R8.1
- no-connect marks 0 -> 7
Other:
- note added: "Battery Connector 4 pin header"
- note added: "Status LED connector"
- moved on the sheet: C12, C2, C3, C4, D4, D5, J2, J3, Q1, Q2, R10, R4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
